Commit message: my naming convention

File: dual_ur_robotiq_description/urdf/dual_ur_robotiq.urdf.xacro (robot description, xacro)
@@ -14,5 +14,5 @@
       <origin xyz="0 0 1.8" rpy="0 0 ${PI/2}"/>
       <geometry>
-        <mesh filename="package://ur_e_description/meshes/dual_arm_mount.stl" scale="0.03 0.03 0.03" />
+        <mesh filename="package://dual_ur_robotiq_description/meshes/dual_arm_mount.stl" scale="0.03 0.03 0.03" />
       </geometry>
       <material name="DarkGrey">
@@ -23,5 +23,5 @@
       <origin xyz="0 0 1.8" rpy="0 0 ${PI/2}"/>
       <geometry>
-        <mesh filename="package://ur_e_description/meshes/dual_arm_mount.stl" scale="0.03 0.03 0.03" />
+        <mesh filename="package://dual_ur_robotiq_description/meshes/dual_arm_mount.stl" scale="0.03 0.03 0.03" />
       </geometry>
     </collision>
@@ -36,7 +36,7 @@
 <!-- (1) UR5 (extracted from "ur_description/ur5_upload.launch" from "universal_robot" package-->
   <!-- common stuff -->
-  <xacro:include filename="$(find ur_e_description)/urdf/common.gazebo.xacro" />
+  <xacro:include filename="$(find dual_ur_robotiq_description)/urdf/common.gazebo.xacro" />
   <!-- ur5e -->
-  <xacro:include filename="$(find ur_e_description)/urdf/ur5e.urdf.xacro" />
+  <xacro:include filename="$(find dual_ur_robotiq_description)/urdf/ur5e.urdf.xacro" />
   <!-- left arm -->
   <xacro:ur5e_robot prefix="left_" joint_limited="false" transmission_hw_interface="$(arg transmission_hw_interface)"/>

File: dual_ur_robotiq_description/urdf/ur5e.urdf.xacro (robot description, xacro)
@@ -1,6 +1,6 @@
 <?xml version="1.0"?>
 <robot xmlns:xacro="http://ros.org/wiki/xacro">
-  <xacro:include filename="$(find ur_e_description)/urdf/ur.transmission.xacro" />
-  <xacro:include filename="$(find ur_e_description)/urdf/ur.gazebo.xacro" />
+  <xacro:include filename="$(find dual_ur_robotiq_description)/urdf/ur.transmission.xacro" />
+  <xacro:include filename="$(find dual_ur_robotiq_description)/urdf/ur.gazebo.xacro" />
   <xacro:macro name="cylinder_inertial" params="radius length mass *origin">
     <inertial>
@@ -80,13 +80,13 @@
       <visual>
         <geometry>
-          <mesh filename="package://ur_e_description/meshes/ur5e/visual/base.dae" />
-        </geometry>
-        <material name="LightGrey">
-          <color rgba="0.7 0.7 0.7 1.0"/>
-        </material>
-      </visual>
-      <collision>
-        <geometry>
-          <mesh filename="package://ur_e_description/meshes/ur5e/collision/base.stl" />
+          <mesh filename="package://dual_ur_robotiq_description/meshes/ur5e/visual/base.dae" />
+        </geometry>
+        <material name="LightGrey">
+          <color rgba="0.7 0.7 0.7 1.0"/>
+        </material>
+      </visual>
+      <collision>
+        <geometry>
+          <mesh filename="package://dual_ur_robotiq_description/meshes/ur5e/collision/base.stl" />
         </geometry>
       </collision>
@@ -117,13 +117,13 @@
       <visual>
         <geometry>
-          <mesh filename="package://ur_e_description/meshes/ur5e/visual/shoulder.dae" />
-        </geometry>
-        <material name="LightGrey">
-          <color rgba="0.7 0.7 0.7 1.0"/>
-        </material>
-      </visual>
-      <collision>
-        <geometry>
-          <mesh filename="package://ur_e_description/meshes/ur5e/collision/shoulder.stl" />
+          <mesh filename="package://dual_ur_robotiq_description/meshes/ur5e/visual/shoulder.dae" />
+        </geometry>
+        <material name="LightGrey">
+          <color rgba="0.7 0.7 0.7 1.0"/>
+        </material>
+      </visual>
+      <collision>
+        <geometry>
+          <mesh filename="package://dual_ur_robotiq_description/meshes/ur5e/collision/shoulder.stl" />
         </geometry>
       </collision>
@@ -154,13 +154,13 @@
       <visual>
         <geometry>
-          <mesh filename="package://ur_e_description/meshes/ur5e/visual/upperarm.dae" />
-        </geometry>
-        <material name="LightGrey">
-          <color rgba="0.7 0.7 0.7 1.0"/>
-        </material>
-      </visual>
-      <collision>
-        <geometry>
-          <mesh filename="package://ur_e_description/meshes/ur5e/collision/upperarm.stl" />
+          <mesh filename="package://dual_ur_robotiq_description/meshes/ur5e/visual/upperarm.dae" />
+        </geometry>
+        <material name="LightGrey">
+          <color rgba="0.7 0.7 0.7 1.0"/>
+        </material>
+      </visual>
+      <collision>
+        <geometry>
+          <mesh filename="package://dual_ur_robotiq_description/meshes/ur5e/collision/upperarm.stl" />
         </geometry>
       </collision>
@@ -191,13 +191,13 @@
       <visual>
         <geometry>
-          <mesh filename="package://ur_e_description/meshes/ur5e/visual/forearm.dae" />
-        </geometry>
-        <material name="LightGrey">
-          <color rgba="0.7 0.7 0.7 1.0"/>
-        </material>
-      </visual>
-      <collision>
-        <geometry>
-          <mesh filename="package://ur_e_description/meshes/ur5e/collision/forearm.stl" />
+          <mesh filename="package://dual_ur_robotiq_description/meshes/ur5e/visual/forearm.dae" />
+        </geometry>
+        <material name="LightGrey">
+          <color rgba="0.7 0.7 0.7 1.0"/>
+        </material>
+      </visual>
+      <collision>
+        <geometry>
+          <mesh filename="package://dual_ur_robotiq_description/meshes/ur5e/collision/forearm.stl" />
         </geometry>
       </collision>
@@ -228,13 +228,13 @@
       <visual>
         <geometry>
-          <mesh filename="package://ur_e_description/meshes/ur5e/visual/wrist1.dae" />
-        </geometry>
-        <material name="LightGrey">
-          <color rgba="0.7 0.7 0.7 1.0"/>
-        </material>
-      </visual>
-      <collision>
-        <geometry>
-          <mesh filename="package://ur_e_description/meshes/ur5e/collision/wrist1.stl" />
+          <mesh filename="package://dual_ur_robotiq_description/meshes/ur5e/visual/wrist1.dae" />
+        </geometry>
+        <material name="LightGrey">
+          <color rgba="0.7 0.7 0.7 1.0"/>
+        </material>
+      </visual>
+      <collision>
+        <geometry>
+          <mesh filename="package://dual_ur_robotiq_description/meshes/ur5e/collision/wrist1.stl" />
         </geometry>
       </collision>
@@ -265,13 +265,13 @@
       <visual>
         <geometry>
-          <mesh filename="package://ur_e_description/meshes/ur5e/visual/wrist2.dae" />
-        </geometry>
-        <material name="LightGrey">
-          <color rgba="0.7 0.7 0.7 1.0"/>
-        </material>
-      </visual>
-      <collision>
-        <geometry>
-          <mesh filename="package://ur_e_description/meshes/ur5e/collision/wrist2.stl" />
+          <mesh filename="package://dual_ur_robotiq_description/meshes/ur5e/visual/wrist2.dae" />
+        </geometry>
+        <material name="LightGrey">
+          <color rgba="0.7 0.7 0.7 1.0"/>
+        </material>
+      </visual>
+      <collision>
+        <geometry>
+          <mesh filename="package://dual_ur_robotiq_description/meshes/ur5e/collision/wrist2.stl" />
         </geometry>
       </collision>
@@ -302,13 +302,13 @@
       <visual>
         <geometry>
-          <mesh filename="package://ur_e_description/meshes/ur5e/visual/wrist3.dae" />
-        </geometry>
-        <material name="LightGrey">
-          <color rgba="0.7 0.7 0.7 1.0"/>
-        </material>
-      </visual>
-      <collision>
-        <geometry>
-          <mesh filename="package://ur_e_description/meshes/ur5e/collision/wrist3.stl" />
+          <mesh filename="package://dual_ur_robotiq_description/meshes/ur5e/visual/wrist3.dae" />
+        </geometry>
+        <material name="LightGrey">
+          <color rgba="0.7 0.7 0.7 1.0"/>
+        </material>
+      </visual>
+      <collision>
+        <geometry>
+          <mesh filename="package://dual_ur_robotiq_description/meshes/ur5e/collision/wrist3.stl" />
         </geometry>
       </collision>

File: dual_ur_robotiq_description/urdf/ur5e_joint_limited_robot.urdf.xacro (robot description, xacro)
@@ -3,7 +3,7 @@
        name="ur5e" >
   <!-- common stuff -->
-  <xacro:include filename="$(find ur_e_description)/urdf/common.gazebo.xacro" />
+  <xacro:include filename="$(find dual_ur_robotiq_description)/urdf/common.gazebo.xacro" />
   <!-- ur5e -->
-  <xacro:include filename="$(find ur_e_description)/urdf/ur5e.urdf.xacro" />
+  <xacro:include filename="$(find dual_ur_robotiq_description)/urdf/ur5e.urdf.xacro" />
   <!-- arm -->
   <xacro:ur5e_robot prefix="" joint_limited="true"

File: dual_ur_robotiq_description/urdf/ur5e_robot.urdf.xacro (robot description, xacro)
@@ -3,7 +3,7 @@
        name="ur5e" >
   <!-- common stuff -->
-  <xacro:include filename="$(find ur_e_description)/urdf/common.gazebo.xacro" />
+  <xacro:include filename="$(find dual_ur_robotiq_description)/urdf/common.gazebo.xacro" />
   <!-- ur5e -->
-  <xacro:include filename="$(find ur_e_description)/urdf/ur5e.urdf.xacro" />
+  <xacro:include filename="$(find dual_ur_robotiq_description)/urdf/ur5e.urdf.xacro" />
   <!-- arm -->
   <xacro:ur5e_robot prefix="" joint_limited="false"/>
