Commit message: pick place example

File: dual_ur_robotiq_description/urdf/robot.urdf.xacro (robot description, xacro)
@@ -39,16 +39,16 @@
   <!-- ur5e -->
   <xacro:include filename="$(find dual_ur_robotiq_description)/urdf/ur5e.urdf.xacro" />
+  <!-- right arm -->
+  <xacro:ur5e_robot prefix="right_" joint_limited="false" transmission_hw_interface="$(arg transmission_hw_interface)"/>
   <!-- left arm -->
   <xacro:ur5e_robot prefix="left_" joint_limited="false" transmission_hw_interface="$(arg transmission_hw_interface)"/>
-  <!-- right arm -->
-  <xacro:ur5e_robot prefix="right_" joint_limited="false" transmission_hw_interface="$(arg transmission_hw_interface)"/>
+  <joint name="right_arm_joint" type="fixed">
+    <parent link="stand" />
+    <child link = "right_base_link" />
+    <origin xyz="0 0.35 1.8" rpy="${PI/4*3} 0 ${PI}" />
+  </joint>
   <joint name="left_arm_joint" type="fixed">
     <parent link="stand" />
     <child link = "left_base_link" />
-    <origin xyz="0 0.35 1.8" rpy="${PI/4*3} 0 ${PI}" />
-  </joint>
-  <joint name="right_arm_joint" type="fixed">
-    <parent link="stand" />
-    <child link = "right_base_link" />
     <origin xyz="0 -0.35 1.8" rpy="${PI/4*3} 0 0" />
   </joint>
@@ -56,8 +56,13 @@
   <!-- robotieq 3f gripper -->
   <xacro:include filename="$(find robotiq_3f_gripper_visualization)/cfg/robotiq-3f-gripper_articulated_macro.xacro" />
+  <!-- right gripper -->
+  <xacro:robotiq-3f-gripper_articulated prefix="right_"/>
   <!-- left gripper -->
   <xacro:robotiq-3f-gripper_articulated prefix="left_"/>
-  <!-- right gripper -->
-  <xacro:robotiq-3f-gripper_articulated prefix="right_"/>
+  <joint name="right_gripper_joint" type="fixed">
+    <parent link="right_ee_link" />
+    <child link = "right_palm" />
+    <origin xyz="0.05 0 0" rpy="0 ${PI/4*3} -${PI/2}" />
+  </joint>
   <joint name="left_gripper_joint" type="fixed">
     <parent link="left_ee_link" />
@@ -65,8 +70,3 @@
     <origin xyz="0.05 0 0" rpy="0 ${PI/4*3} -${PI/2}" />
   </joint>
-  <joint name="right_gripper_joint" type="fixed">
-    <parent link="right_ee_link" />
-    <child link = "right_palm" />
-    <origin xyz="0.05 0 0" rpy="0 ${PI/4*3} -${PI/2}" />
-  </joint>
 </robot>

File: ur_e_description/urdf/dual_ur5e_robot.urdf.xacro (robot description, xacro)
@@ -9,5 +9,5 @@
       <origin xyz="0 0 1.8" rpy="0 0 ${PI/2}"/>
       <geometry>
-        <mesh filename="package://ur_e_description/meshes/dual_arm_mount.stl" scale="0.03 0.03 0.03" />
+        <mesh filename="package://dual_ur_robotiq_description/meshes/dual_arm_mount.stl" scale="0.03 0.03 0.03" />
       </geometry>
       <material name="DarkGrey">
@@ -18,5 +18,5 @@
       <origin xyz="0 0 1.8" rpy="0 0 ${PI/2}"/>
       <geometry>
-        <mesh filename="package://ur_e_description/meshes/dual_arm_mount.stl" scale="0.03 0.03 0.03" />
+        <mesh filename="package://dual_ur_robotiq_description/meshes/dual_arm_mount.stl" scale="0.03 0.03 0.03" />
       </geometry>
     </collision>
@@ -31,7 +31,7 @@
 <!-- (1) UR5 (extracted from "ur_description/ur5_upload.launch" from "universal_robot" package-->
   <!-- common stuff -->
-  <xacro:include filename="$(find ur_e_description)/urdf/common.gazebo.xacro" />
+  <xacro:include filename="$(find dual_ur_robotiq_description)/urdf/common.gazebo.xacro" />
   <!-- ur5e -->
-  <xacro:include filename="$(find ur_e_description)/urdf/ur5e.urdf.xacro" />
+  <xacro:include filename="$(find dual_ur_robotiq_description)/urdf/ur5e.urdf.xacro" />
   <!-- left arm -->
   <xacro:ur5e_robot prefix="left_" joint_limited="false" transmission_hw_interface="$(arg transmission_hw_interface)"/>

Commit message: Fix real robot positional error

File: dual_ur_robotiq_description/urdf/robot.urdf.xacro (robot description, xacro)
@@ -46,10 +46,10 @@
     <parent link="stand" />
     <child link = "right_base_link" />
-    <origin xyz="0 0.35 1.8" rpy="${PI/4*3} 0 ${PI}" />
+    <origin xyz="0 0.35 1.8" rpy="${PI/4*3} 0.028 ${PI}" />
   </joint>
   <joint name="left_arm_joint" type="fixed">
     <parent link="stand" />
     <child link = "left_base_link" />
-    <origin xyz="0 -0.35 1.8" rpy="${PI/4*3} 0 0" />
+    <origin xyz="0 -0.35 1.803" rpy="${(PI/4*3)+0.003} -0.005 0" />
   </joint>
 <!-- (2) Robotiq 3-finger gripper (Right Hand)-->
@@ -63,5 +63,5 @@
     <parent link="right_ee_link" />
     <child link = "right_palm" />
-    <origin xyz="0.05 0 0" rpy="0 ${PI/4*3} -${PI/2}" />
+    <origin xyz="0.05 0 0" rpy="0 -${PI/4} -${PI/2}" />
   </joint>
   <joint name="left_gripper_joint" type="fixed">

Commit message: Update robot description

File: dual_ur_robotiq_description/urdf/robot.urdf.xacro (robot description, xacro)
@@ -46,10 +46,13 @@
     <parent link="stand" />
     <child link = "right_base_link" />
-    <origin xyz="0 0.35 1.8" rpy="${PI/4*3} 0.028 ${PI}" />
+    <!--origin xyz="0 0.3 1.8" rpy="${PI/4*3} 0.028 ${PI}" /-->
+    <origin xyz="0 0.305 1.65" rpy="${PI/4*3} 0 ${PI}" />
   </joint>
   <joint name="left_arm_joint" type="fixed">
     <parent link="stand" />
     <child link = "left_base_link" />
-    <origin xyz="0 -0.35 1.803" rpy="${(PI/4*3)+0.003} -0.005 0" />
+    <!--origin xyz="0 -0.3 1.803" rpy="${(PI/4*3)+0.003} -0.005 0" /-->
+    <origin xyz="-0.01 -0.305 1.65" rpy="${PI/4*3} 0 0" />
+    <!-- origin xyz="0 -0.3 1.65" rpy="${PI/4*3} 0 0" /-->
   </joint>
 <!-- (2) Robotiq 3-finger gripper (Right Hand)-->
@@ -63,5 +66,5 @@
     <parent link="right_ee_link" />
     <child link = "right_palm" />
-    <origin xyz="0.05 0 0" rpy="0 -${PI/4} -${PI/2}" />
+    <origin xyz="0.05 0 0" rpy="0 ${PI/4*3} -${PI/2}" />
   </joint>
   <joint name="left_gripper_joint" type="fixed">

File: dual_ur_robotiq_description/urdf/ur5e_joint_limited_robot.urdf.xacro (robot description, xacro)
@@ -13,5 +13,5 @@
     wrist_1_lower_limit="${-pi}" wrist_1_upper_limit="${pi}"
     wrist_2_lower_limit="${-pi}" wrist_2_upper_limit="${pi}"
-    wrist_3_lower_limit="${-pi}" wrist_3_upper_limit="${pi}"
+    wrist_3_lower_limit="${-pi}/2" wrist_3_upper_limit="${pi}/2"
   />
   <link name="world" />
