Commit message: minor change

File: ur_description/urdf/dual_ur5e.urdf.xacro (robot description, xacro)
@@ -4,7 +4,7 @@
   <xacro:arg name="transmission_hw_interface" default="hardware_interface/PositionJointInterface"/>
   <!-- common stuff -->
-  <xacro:include filename="$(find ur_e_description)/urdf/common.gazebo.xacro" />
+  <xacro:include filename="$(find dual_ur_robotiq_description)/urdf/common.gazebo.xacro" />
   <!-- ur5e -->
-  <xacro:include filename="$(find ur_e_description)/urdf/ur5e.urdf.xacro" />
+  <xacro:include filename="$(find dual_ur_robotiq_description)/urdf/ur5e.urdf.xacro" />
   <!-- left arm -->
   <xacro:ur5e_robot prefix="left_" joint_limited="false" transmission_hw_interface="$(arg transmission_hw_interface)"/>
@@ -15,5 +15,5 @@
       <origin xyz="0 0 1.6" rpy="0 0 ${PI/2}"/>
       <geometry>
-        <mesh filename="package://ur_e_description/meshes/dual_arm_mount.stl" scale="0.03 0.03 0.03" />
+        <mesh filename="package://dual_ur_robotiq_description/meshes/dual_arm_mount.stl" scale="0.03 0.03 0.03" />
       </geometry>
       <material name="DarkGrey">
@@ -24,5 +24,5 @@
       <origin xyz="0 0 1.6" rpy="0 0 ${PI/2}"/>
       <geometry>
-        <mesh filename="package://ur_e_description/meshes/dual_arm_mount.stl" scale="0.03 0.03 0.03" />
+        <mesh filename="package://dual_ur_robotiq_description/meshes/dual_arm_mount.stl" scale="0.03 0.03 0.03" />
       </geometry>
     </collision>
